File: DRC-SerialSVMD2026.ver.0.2.1.kicad_sch (KiCad schematic)
At the start: 32 parts, among them J1 USB, J11 SerialServo1, J12 SerialServo2, J7 CAN, J8 CAN, J9 +BATT, SW4 SW_SPDT, SW6 SW_DPDT_x2, U1 RT9080-33GJ5, U2 78L05G-AB3-R, U6 SN65HVD230

Commit message: Update board design and PCBA manufacturing files
Parts:
- D2: value 1N4148WT -> 1N4148W
Changed lines of the file:
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@@
 			)
 		)
-		(property "Value" "1N4148WT"
+		(property "Value" "1N4148W"
 			(at 133.096 171.45 0)
 			(effects
