File: STSServoDrive.kicad_sch (KiCad schematic)
At the start: 10 parts, among them Q1 MMBT3906, U3 Si8621EC-B-IS, U4 MAX485E

Commit message: Update board design and PCBA manufacturing files
Parts:
- R9: value 10k -> 5.1k
Changed lines of the file:
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@@
 			)
 		)
-		(property "Value" "10k"
+		(property "Value" "5.1k"
 			(at 152.4 110.4899 0)
 			(effects
