File: DRC-SerialSVMD2026.ver.0.2.1.kicad_pcb (KiCad board)
At the start: 2 copper layers, 60 x 45 mm, 81 parts, among them J1 USB, J11 SerialServo1, J12 SerialServo2, J16 USB_C, J7 CAN, J8 CAN, J9 +BATT, Q1 MMBT3906, SW1 BOOT, SW2 RESET, SW3 SW_DIP_x02, SW4 SW_SPDT, SW6 SW_DPDT_x2, U1 RT9080-33GJ5, U2 78L05G-AB3-R, U3 Si8621EC-B-IS, U4 MAX485E, U5 RP2354A, U6 SN65HVD230, U7 CH340E, Y1 12MHz_ABM8-272-T3

Commit message: Update board design and PCBA manufacturing files
Parts:
- D2: value 1N4148WT -> 1N4148W
- R9: value 10k -> 5.1k
- moved C20 1.68 mm to (17.5, 33.8)
- moved Y1 1.66 mm to (15.4, 34.8)
- moved C21 1.46 mm to (17.5, 35.8)
- moved L1 0.37 mm to (32.6, 37.4)
- moved J11 0.07 mm to (29.3, 8.99)
Routing:
- net Net-(U5-XIN): track 9.80 -> 7.33 mm
- net Net-(C21-Pad1): track 4.43 -> 2.78 mm
- net Net-(U5-RUN): track 6.30 -> 5.25 mm
- net GND: track 0.00 -> 0.21 mm, vias 17 -> 57
- net GNDPWR: vias 6 -> 18
- net +BATT: vias 5 -> 10

Commit message: Update PCB layout
Other:
- board text added: "USB Servo"
- board text added: "USB-MCU"
Changed lines of the file:
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@@
 		(tags "USB C Type-C Receptacle SMD USB 2.0 16P 16C USB4105-15-A USB4105-15-A-060 USB4105-15-A-120 USB4105-GF-A USB4105-GF-A-060 USB4105-GF-A-120")
 		(property "Reference" "J16"
-			(at 0 -5.5 180)
+			(at 0 0.0082 180)
 			(unlocked yes)
 			(layer "F.SilkS")
@@
 		(tags "USB C Type-C Receptacle SMD USB 2.0 16P 16C USB4105-15-A USB4105-15-A-060 USB4105-15-A-120 USB4105-GF-A USB4105-GF-A-060 USB4105-GF-A-120")
 		(property "Reference" "J1"
-			(at 0 -5.5 0)
+			(at 0 0 0)
 			(unlocked yes)
 			(layer "F.SilkS")
@@
 		(tags "TSOT-23-5 Hand-soldering")
 		(property "Reference" "U1"
-			(at 2.4048 -2.3876 0)
+			(at 0 0 0)
 			(layer "F.SilkS")
 			(effects
@@
 		)
 	)
+	(gr_text "USB\nServo"
+		(at 47.371 8.763 180)
+		(layer "F.SilkS")
+		(effects
+			(font
+				(size 1 1)
+				(thickness 0.1)
+			)
+			(justify left bottom)
+		)
+	)
 	(gr_text "DRC-SerialSVMD2026"
 		(at 7.7216 42.7228 0)
@@
 		)
 	)
+	(gr_text "USB-MCU"
+		(at 39.116 36.322 0)
+		(layer "F.SilkS")
+		(effects
+			(font
+				(size 1 1)
+				(thickness 0.1)
+			)
+			(justify left bottom)
+		)
+	)
 	(segment
 		(start 51.7328 11.2668)
@@
 	)
 	(segment
-		(start 48.039178 8.1452)
-		(end 46.766 9.418378)
+		(start 47.659106 8.419165)
+		(end 47.765213 8.419165)
 		(width 0.25)
 		(layer "F.Cu")
@@
 	)
 	(segment
-		(start 46.766 9.418378)
-		(end 46.366145 9.418378)
+		(start 48.248 7.936378)
+		(end 48.248 7.2442)
 		(width 0.25)
 		(layer "F.Cu")
@@
 	)
 	(segment
-		(start 48.248 7.936378)
-		(end 48.248 7.2442)
+		(start 47.248 7.888378)
+		(end 47.504822 8.1452)
 		(width 0.25)
 		(layer "F.Cu")
@@
 	)
 	(segment
-		(start 47.248 7.888378)
-		(end 47.504822 8.1452)
+		(start 47.765213 8.419165)
+		(end 48.039178 8.1452)
 		(width 0.25)
 		(layer "F.Cu")
@@
 	)
 	(via
-		(at 46.366145 9.418378)
+		(at 47.659106 8.419165)
 		(size 0.8)
 		(drill 0.4)
@@
 	)
 	(segment
-		(start 44.747122 9.418378)
-		(end 46.366145 9.418378)
+		(start 47.659106 8.419165)
+		(end 46.659893 9.418378)
 		(width 0.25)
 		(layer "B.Cu")
@@
 	)
 	(segment
-		(start 44.569 11.176)
+		(start 46.659893 9.418378)
+		(end 44.747122 9.418378)
+		(width 0.25)
+		(layer "B.Cu")
+		(net 78)
+	)
+	(segment
+		(start 44.747122 9.418378)
 		(end 44.569 9.5965)
 		(width 0.25)
@@
 	(segment
 		(start 44.569 9.5965)
-		(end 44.747122 9.418378)
+		(end 44.569 11.176)
 		(width 0.25)
 		(layer "B.Cu")
@@
 			(pts
 				(xy 27.178 36.2204) (xy 28.3464 36.2204) (xy 28.8544 36.0172) (xy 30.8864 36.0172) (xy 31.739 36.2776)
-				(xy 33.539 36.2776) (xy 33.539 37.1856) (xy 33.539 37.1856) (xy 31.75 37.1856) (xy 31.4452 37.2872)
-				(xy 30.4292 37.2872) (xy 30.4292 36.4236) (xy 27.4059 36.4236) (xy 27.178 36.4236)
+				(xy 33.539 36.2776) (xy 33.539 37.1856) (xy 31.75 37.1856) (xy 31.4452 37.2872) (xy 30.4292 37.2872)
+				(xy 30.4292 36.4236) (xy 27.4059 36.4236) (xy 27.178 36.4236)
 			)
 		)
